File: Hardware/Cabina360/Cabina360.kicad_pcb (KiCad board)
At the start: 2 copper layers, 66 x 51.7 mm, 47 parts, among them J1 USB_B_Micro, M1 Left, Q1 DMG2301L, Q4 MBT3904DW1, Q5 DMG3406L, SW2 Reset, SW3 Boot, U2 AP2112K-3.3, U3 ESP32-WROOM-32, U7 CH340C

Commit message: ft!: Actualización Sistema Electronico
Parts:
- removed C17: 3.3nF, Capacitor_SMD:C_0805_2012Metric
- removed D9: LED_RGBK, LED_SMD:LED_RGB_5050-6
- removed H3: MountingHole, MountingHole:MountingHole_3.2mm_M3_ISO14580_Pad_TopBottom
- removed M1: Left, Connector_JST:JST_EH_S2B-EH_1x02_P2.50mm_Horizontal
- removed R29, R30, R31: 1K, Resistor_SMD:R_0805_2012Metric
- removed Serial1: 5V RX TX GND, Connector_PinHeader_2.54mm:PinHeader_1x04_P2.54mm_Vertical
- added 5V_ALIM1: 5V GND, TerminalBlock:TerminalBlock_bornier-2_P5.08mm, F.Cu at (76.4, 143.5)
- added BORNERAM1: MOTOR+ MOTOR-, TerminalBlock:TerminalBlock_bornier-2_P5.08mm, F.Cu at (92.1, 108.8)
- added C3: 10uF, Capacitor_THT:CP_Radial_D8.0mm_P3.50mm, F.Cu at (102.7, 107.2)
- added DRIVER_STEP_MOTOR1: Pololu_Breakout_A4988, Module:Pololu_Breakout-16_15.2x20.3mm, F.Cu at (92.5, 117.0)
- added POWE_MOTOR1: PINES, Connector_PinHeader_2.54mm:PinHeader_1x05_P2.54mm_Horizontal, F.Cu at (108.8, 141.3)
- added R5: 10K, Resistor_SMD:R_0805_2012Metric, F.Cu at (119.1, 135.8)
- added SLIPRING1: PINES, TerminalBlock:TerminalBlock_bornier-5_P5.08mm, F.Cu at (76.5, 116.3)
- added SW1: SW_DPDT_x2, Button_Switch_THT:SW_CuK_OS102011MA1QN1_SPDT_Angled, F.Cu at (86.5, 145.2)
- J1: value USB_B_Micro -> USB_C_Receptacle_USB2.0
- moved BZ1 69.6 mm to (157.9, 120.0), turned to -90 degrees
- moved R33 66.5 mm to (151.3, 123.9), turned to 0 degrees
- moved Q5 63.5 mm to (151.3, 121.0), turned to 90 degrees
- moved D8 60.6 mm to (151.2, 118.1), turned to 180 degrees
- moved C2 58.9 mm to (151.3, 116.2), turned to 0 degrees
- moved C1 57.1 mm to (151.3, 114.1), turned to 180 degrees
- moved D1 51.9 mm to (128.9, 147.4), turned to 0 degrees
- moved R4 51.1 mm to (131.7, 144.3), turned to -90 degrees
- moved R3 50.3 mm to (136.9, 146.3), turned to -90 degrees
- moved C7 49.2 mm to (129.7, 144.3), turned to 90 degrees
- moved Q1 49.1 mm to (124.5, 147.9), turned to 180 degrees
- moved R2 47.3 mm to (127.5, 144.3), turned to 90 degrees
- moved R1 46.3 mm to (140.7, 146.4), turned to -90 degrees
- moved U2 44.7 mm to (124.3, 144.3), turned to 180 degrees
- moved C5 42.5 mm to (121.3, 144.3), turned to 90 degrees
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Connections:
- net /Right renamed /IO15
- J1 pad 1: VBUS -> (no net)
- J1 pad 2: /D+ -> (no net)
- J1 pad 3: /D- -> (no net)
- J1 pad 4: unconnected-(J1-Pad4) -> (no net)
- J1 pad 5: GND -> (no net)
- J1 pad 6: Net-(J1-Pad6) -> (no net)
- U3 pad 10: /PWM_IN1A -> /DIR
- U3 pad 11: /PWM_IN2A -> /STEP
- U3 pad 13: /Left -> /F_CARRERA
- U3 pad 14: /Front -> /PWM
- U3 pad 16: /Back -> /LPWM
- U3 pad 24: /G_led -> /RPWM
- U3 pad 30: /PWM_IN1B -> /G_led
Routing:
- net +3V3: track 42.2 -> 164.9 mm, vias 0 -> 5
- net GND: track 76.0 -> 141.1 mm, vias 2 -> 6
- net /F_CARRERA: track 0.00 -> 49.2 mm
- net EN: track 0.00 -> 46.2 mm, vias 0 -> 2
- net +BATT: track 0.00 -> 45.0 mm
- net /VMOT: track 0.00 -> 44.6 mm
- net /RPWM: track 0.00 -> 38.2 mm, vias 0 -> 1
- net /B_led: track 36.7 -> 0.00 mm
- net /PWM: track 0.00 -> 30.4 mm, vias 0 -> 1
- net /LPWM: track 0.00 -> 29.7 mm, vias 0 -> 1
- net VBUS: track 80.1 -> 50.6 mm
- net /DIR: track 0.00 -> 26.6 mm, vias 0 -> 1
- net /STEP: track 0.00 -> 26.1 mm, vias 0 -> 1
- net Net-(DRIVER_STEP_MOTOR1-Pad3): track 0.00 -> 18.4 mm
- net Net-(DRIVER_STEP_MOTOR1-Pad4): track 0.00 -> 17.3 mm
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Other:
- board size 66 x 51.7 mm -> 97.9 x 51.8 mm
